File: Project/tinyv pcb FFC.kicad_sch (KiCad schematic)
At the start: 102 parts, among them J1 JST SH, J2 Pico EZmate, J3 Conn_01x03_Socket, J4 Conn_01x10_Socket, J7 Conn_01x10_Socket, Q1 2N7002, SW1 RST, U1 MCP1700x-330xxTT, U3 STM32F072C8Tx

Commit message: fresh gerbers
Connections:
- net underglow: now also U3.17 (PA7); no longer U3.21 (PB10)
- no-connect marks 7 -> 22
Changed lines of the file:
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@@
   (junction (at 144.78 93.98) (diameter 0) (color 0 0 0 0)
   )
+  (no_connect (at 256.54 96.52))
+  (no_connect (at 223.52 86.36))
+  (no_connect (at 256.54 60.96))
+  (no_connect (at 223.52 66.04))
+  (no_connect (at 223.52 91.44))
   (no_connect (at 26.67 134.62))
   (no_connect (at 223.52 55.88))
+  (no_connect (at 223.52 63.5))
+  (no_connect (at 256.54 76.2))
   (no_connect (at 49.53 121.92))
+  (no_connect (at 223.52 88.9))
   (no_connect (at 223.52 50.8))
   (no_connect (at 256.54 93.98))
   (no_connect (at 223.52 53.34))
+  (no_connect (at 256.54 63.5))
+  (no_connect (at 223.52 45.72))
+  (no_connect (at 256.54 66.04))
+  (no_connect (at 223.52 60.96))
   (no_connect (at 256.54 73.66))
+  (no_connect (at 223.52 99.06))
+  (no_connect (at 223.52 43.18))
+  (no_connect (at 256.54 86.36))
   (wire (pts (xy 49.53 167.64) (xy 49.53 168.91))
     (stroke (width 0) (type default))
@@
     )
   )
-  (global_label "underglow" (shape input) (at 223.52 86.36 180) (fields_autoplaced)
-    (effects (font (size 1.27 1.27)) (justify right))
-    (property "Intersheetrefs" "${INTERSHEET_REFS}" (at 210.9987 86.36 0)
-      (effects (font (size 1.27 1.27)) (justify right) hide)
-    )
-  )
+  (global_label "underglow" (shape input) (at 256.54 78.74 0) (fields_autoplaced)
+    (effects (font (size 1.27 1.27)) (justify left))
+    (property "Intersheetrefs" "${INTERSHEET_REFS}" (at 269.0613 78.74 0)
+      (effects (font (size 1.27 1.27)) (justify left) hide)
+    )
+  )
